Commit message: changed name to prefix in description

File: description/urdf/scanCONTROL_2600-100.urdf.xacro (robot description, xacro)
@@ -5,5 +5,5 @@
   <link name="base_link"/>
 <!-- sensor -->
-  <xacro:scanCONTROL_2600-100 name="scanCONTROL_2600-100" parent="base_link">
+  <xacro:scanCONTROL_2600-100 prefix="scanCONTROL_2600-100" parent="base_link">
       <origin xyz="0 0 0" rpy="0 0 0" />
   </xacro:scanCONTROL_2600-100>

File: description/urdf/scanCONTROL_2600-100_macro.urdf.xacro (robot description, xacro)
@@ -1,11 +1,11 @@
 <?xml version="1.0"?>
 <robot xmlns:xacro="http://www.ros.org/wiki/xacro">
-    <xacro:macro name="scanCONTROL_2600-100" params="parent name *origin">
-        <joint name="${name}_sensor_joint" type="fixed">
+    <xacro:macro name="scanCONTROL_2600-100" params="parent prefix *origin">
+        <joint name="${prefix}_sensor_joint" type="fixed">
             <xacro:insert_block name="origin" />
             <parent link="${parent}"/>
-            <child link="${name}_sensor_link" />
+            <child link="${prefix}_sensor_link" />
         </joint>
-        <link name="${name}_sensor_link">
+        <link name="${prefix}_sensor_link">
             <inertial>
                 <mass value="0.01" />
