Commit message: Changed link name

File: description/urdf/scanCONTROL_2600-100_macro.urdf.xacro (robot description, xacro)
@@ -2,10 +2,10 @@
 <robot xmlns:xacro="http://www.ros.org/wiki/xacro">
     <xacro:macro name="scanCONTROL_2600-100" params="parent prefix *origin">
-        <joint name="${prefix}_sensor_joint" type="fixed">
+        <joint name="${prefix}scanner_joint" type="fixed">
             <xacro:insert_block name="origin" />
             <parent link="${parent}"/>
-            <child link="${prefix}_sensor_link" />
+            <child link="${prefix}scanner_link" />
         </joint>
-        <link name="${prefix}_sensor_link">
+        <link name="${prefix}scanner_link">
             <inertial>
                 <mass value="0.01" />

Commit message: added scanner_laser_link and calibrated it

File: description/urdf/scanCONTROL_2600-100_macro.urdf.xacro (robot description, xacro)
@@ -24,4 +24,15 @@
             </collision>
         </link>
+        <!--<joint name="${prefix}scanner_laser_joint" type="fixed">
+            <origin xyz="0 0 0" rpy="0 0 ${pi}" />
+            <parent link="${prefix}scanner_link"/>
+            <child link="${prefix}scanner_laser_link" />
+        </joint>-->
+        <joint name="${prefix}scanner_laser_joint" type="fixed">
+            <origin xyz="0.0383464 0.109996 0.135064" rpy="${radians(0.242595)} ${radians(0.0646638)} ${radians(-92.129)}" />
+            <parent link="tool0"/>
+            <child link="${prefix}scanner_laser_link" />
+        </joint>
+        <link name="${prefix}scanner_laser_link" />
   </xacro:macro>
 </robot>
